File: 75thruhole.sch (KiCad schematic (older format))
At the start: 24 parts, among them K1 KEYSW, K2 KEYSW, K3 KEYSW, K4 KEYSW, SW1 SW_PUSH, U1 ATMEGA32U4, X1 XTAL_GND

Commit message: matching
Parts:
- gave numbers to parts that had none: 1
Connections:
- net +5V: now also U1.15 (GND), U1.24 (AVCC), U1.35 (GND), U1.43 (GND)
- net VCC: now also U1.14 (VCC), U1.23 (GND), U1.34 (VCC), U1.44 (AVCC), U1.7 (VBus)
- net col1: now reaches U1.38 (PF5)
- net col1: now also K3.1, K4.1
- net col0: now reaches U1.39 (PF4)
- net col0: now also K1.1, K2.1
- net row1: now reaches U1.40 (PF1)
- net row0: now reaches U1.41 (PF0)
- no-connect marks 0 -> 24
Other:
- moved on the sheet: R1

Commit message: generate pcb
Parts:
- C1, C2, C3, C4, C5, C6, C7, C8: footprint (none) -> Capacitor_SMD:C_0805_2012Metric_Pad1.15x1.40mm_HandSolder
- D1, D2, D3, D4: footprint (none) -> keyboard_parts:D_SOD123_axial
- J1: footprint (none) -> keyboard_parts:USB_miniB_hirose_5S8
- K1, K2, K3, K4: footprint (none) -> keebs:Mx_Alps_100
- R1, R2, R3, R4: footprint (none) -> Resistor_SMD:R_0805_2012Metric_Pad1.15x1.40mm_HandSolder
- SW1: footprint (none) -> Button_Switch_SMD:SW_SPST_TL3342
- U1: footprint (none) -> Package_QFP:TQFP-44_10x10mm_P0.8mm
- X1: footprint (none) -> keyboard_parts:FA-238
Changed lines of the file:
@@
 EESchema Schematic File Version 4
-LIBS:75thruhole-cache
 EELAYER 30 0
 EELAYER END
@@
 F 0 "U1" H 3900 1300 60  0000 C CNN
 F 1 "ATMEGA32U4" H 3925 3731 60  0000 C CNN
-F 2 "" H 3900 2500 60  0001 C CNN
+F 2 "Package_QFP:TQFP-44_10x10mm_P0.8mm" H 3900 2500 60  0001 C CNN
 F 3 "" H 3900 2500 60  0000 C CNN
 	1    3900 2500
@@
 F 0 "X1" H 1850 2950 60  0000 C CNN
 F 1 "XTAL_GND" H 1850 3200 60  0000 C CNN
-F 2 "" H 1850 3050 60  0001 C CNN
+F 2 "keyboard_parts:FA-238" H 1850 3050 60  0001 C CNN
 F 3 "" H 1850 3050 60  0000 C CNN
 	1    1850 3050
@@
 F 0 "C1" H 2150 3350 50  0000 L CNN
 F 1 "22p" H 2150 3150 50  0000 L CNN
-F 2 "" H 2150 3250 50  0001 C CNN
+F 2 "Capacitor_SMD:C_0805_2012Metric_Pad1.15x1.40mm_HandSolder" H 2150 3250 50  0001 C CNN
 F 3 "~" H 2150 3250 50  0001 C CNN
 	1    2150 3250
@@
 F 0 "C2" H 1450 3350 50  0000 L CNN
 F 1 "22p" H 1400 3150 50  0000 L CNN
-F 2 "" H 1550 3250 50  0001 C CNN
+F 2 "Capacitor_SMD:C_0805_2012Metric_Pad1.15x1.40mm_HandSolder" H 1550 3250 50  0001 C CNN
 F 3 "~" H 1550 3250 50  0001 C CNN
 	1    1550 3250
@@
 F 0 "C3" H 1450 1150 50  0000 L CNN
 F 1 "0.1u" H 1450 950 50  0000 L CNN
-F 2 "" H 1400 1050 50  0001 C CNN
+F 2 "Capacitor_SMD:C_0805_2012Metric_Pad1.15x1.40mm_HandSolder" H 1400 1050 50  0001 C CNN
 F 3 "~" H 1400 1050 50  0001 C CNN
 	1    1400 1050
@@
 F 0 "C4" H 1750 1150 50  0000 L CNN
 F 1 "0.1u" H 1750 950 50  0000 L CNN
-F 2 "" H 1700 1050 50  0001 C CNN
+F 2 "Capacitor_SMD:C_0805_2012Metric_Pad1.15x1.40mm_HandSolder" H 1700 1050 50  0001 C CNN
 F 3 "~" H 1700 1050 50  0001 C CNN
 	1    1700 1050
@@
 F 0 "C5" H 2050 1150 50  0000 L CNN
 F 1 "0.1u" H 2050 950 50  0000 L CNN
-F 2 "" H 2000 1050 50  0001 C CNN
+F 2 "Capacitor_SMD:C_0805_2012Metric_Pad1.15x1.40mm_HandSolder" H 2000 1050 50  0001 C CNN
 F 3 "~" H 2000 1050 50  0001 C CNN
 	1    2000 1050
@@
 F 0 "C6" H 2350 1150 50  0000 L CNN
 F 1 "0.1u" H 2350 950 50  0000 L CNN
-F 2 "" H 2300 1050 50  0001 C CNN
+F 2 "Capacitor_SMD:C_0805_2012Metric_Pad1.15x1.40mm_HandSolder" H 2300 1050 50  0001 C CNN
 F 3 "~" H 2300 1050 50  0001 C CNN
 	1    2300 1050
@@
 F 0 "C7" H 2600 1150 50  0000 L CNN
 F 1 "4.7u" H 2650 950 50  0000 L CNN
-F 2 "" H 2600 1050 50  0001 C CNN
+F 2 "Capacitor_SMD:C_0805_2012Metric_Pad1.15x1.40mm_HandSolder" H 2600 1050 50  0001 C CNN
 F 3 "~" H 2600 1050 50  0001 C CNN
 	1    2600 1050
@@
 F 0 "SW1" H 1850 2800 50  0000 C CNN
 F 1 "SW_PUSH" H 1850 2550 50  0000 C CNN
-F 2 "" H 1850 2650 60  0001 C CNN
+F 2 "Button_Switch_SMD:SW_SPST_TL3342" H 1850 2650 60  0001 C CNN
 F 3 "" H 1850 2650 60  0000 C CNN
 	1    1850 2650
@@
 F 0 "R1" V 1750 2400 50  0000 C CNN
 F 1 "10k" V 1850 2400 50  0000 C CNN
-F 2 "" V 1780 2400 50  0001 C CNN
+F 2 "Resistor_SMD:R_0805_2012Metric_Pad1.15x1.40mm_HandSolder" V 1780 2400 50  0001 C CNN
 F 3 "~" H 1850 2400 50  0001 C CNN
 	1    1850 2400
@@
 F 0 "R2" V 5350 2550 50  0000 C CNN
 F 1 "10k" V 5250 2550 50  0000 C CNN
-F 2 "" V 5180 2550 50  0001 C CNN
+F 2 "Resistor_SMD:R_0805_2012Metric_Pad1.15x1.40mm_HandSolder" V 5180 2550 50  0001 C CNN
 F 3 "~" H 5250 2550 50  0001 C CNN
 	1    5250 2550
@@
 F 0 "J1" H 1300 1700 60  0000 C CNN
 F 1 "USB_mini_micro_B" H 1550 1950 60  0001 C CNN
-F 2 "" H 1650 1700 60  0001 C CNN
+F 2 "keyboard_parts:USB_miniB_hirose_5S8" H 1650 1700 60  0001 C CNN
 F 3 "" H 1650 1700 60  0000 C CNN
 	1    1700 1700
@@
 F 0 "R3" V 2500 1600 50  0000 C CNN
 F 1 "22" V 2500 1700 50  0000 C CNN
-F 2 "" V 2430 1650 50  0001 C CNN
+F 2 "Resistor_SMD:R_0805_2012Metric_Pad1.15x1.40mm_HandSolder" V 2430 1650 50  0001 C CNN
 F 3 "~" H 2500 1650 50  0001 C CNN
 	1    2500 1650
@@
 F 0 "R4" V 2500 1700 50  0000 C CNN
 F 1 "22" V 2500 1800 50  0000 C CNN
-F 2 "" V 2430 1750 50  0001 C CNN
+F 2 "Resistor_SMD:R_0805_2012Metric_Pad1.15x1.40mm_HandSolder" V 2430 1750 50  0001 C CNN
 F 3 "~" H 2500 1750 50  0001 C CNN
 	1    2500 1750
@@
 F 0 "C8" V 2700 1850 39  0000 C CNN
 F 1 "1u" V 2700 2050 39  0000 C CNN
-F 2 "" H 2650 1950 50  0001 C CNN
+F 2 "Capacitor_SMD:C_0805_2012Metric_Pad1.15x1.40mm_HandSolder" H 2650 1950 50  0001 C CNN
 F 3 "~" H 2650 1950 50  0001 C CNN
 	1    2650 1950
@@
 F 0 "K1" H 5950 1000 60  0000 C CNN
 F 1 "KEYSW" H 6000 900 60  0001 C CNN
-F 2 "" H 6000 1000 60  0001 C CNN
+F 2 "keebs:Mx_Alps_100" H 6000 1000 60  0001 C CNN
 F 3 "" H 6000 1000 60  0000 C CNN
 	1    6000 1000
@@
 F 0 "K3" H 6650 1000 60  0000 C CNN
 F 1 "KEYSW" H 6700 900 60  0001 C CNN
-F 2 "" H 6700 1000 60  0001 C CNN
+F 2 "keebs:Mx_Alps_100" H 6700 1000 60  0001 C CNN
 F 3 "" H 6700 1000 60  0000 C CNN
 	1    6700 1000
@@
 F 0 "K2" H 5950 1550 60  0000 C CNN
 F 1 "KEYSW" H 6000 1450 60  0001 C CNN
-F 2 "" H 6000 1550 60  0001 C CNN
+F 2 "keebs:Mx_Alps_100" H 6000 1550 60  0001 C CNN
 F 3 "" H 6000 1550 60  0000 C CNN
 	1    6000 1550
@@
 F 0 "K4" H 6650 1550 60  0000 C CNN
 F 1 "KEYSW" H 6700 1450 60  0001 C CNN
-F 2 "" H 6700 1550 60  0001 C CNN
+F 2 "keebs:Mx_Alps_100" H 6700 1550 60  0001 C CNN
 F 3 "" H 6700 1550 60  0000 C CNN
 	1    6700 1550
@@
 F 0 "D1" H 5572 1200 60  0000 R CNN
 F 1 "D" V 5850 1200 60  0001 C CNN
-F 2 "" H 5700 1250 60  0001 C CNN
+F 2 "keyboard_parts:D_SOD123_axial" H 5700 1250 60  0001 C CNN
 F 3 "" H 5700 1250 60  0000 C CNN
 	1    5700 1250
@@
 F 0 "D4" H 6272 1750 60  0000 R CNN
 F 1 "D" V 6550 1750 60  0001 C CNN
-F 2 "" H 6400 1800 60  0001 C CNN
+F 2 "keyboard_parts:D_SOD123_axial" H 6400 1800 60  0001 C CNN
 F 3 "" H 6400 1800 60  0000 C CNN
 	1    6400 1800
@@
 F 0 "D2" H 6272 1200 60  0000 R CNN
 F 1 "D" V 6550 1200 60  0001 C CNN
-F 2 "" H 6400 1250 60  0001 C CNN
+F 2 "keyboard_parts:D_SOD123_axial" H 6400 1250 60  0001 C CNN
 F 3 "" H 6400 1250 60  0000 C CNN
 	1    6400 1250
@@
 F 0 "D3" H 5572 1750 60  0000 R CNN
 F 1 "D" V 5850 1750 60  0001 C CNN
-F 2 "" H 5700 1800 60  0001 C CNN
+F 2 "keyboard_parts:D_SOD123_axial" H 5700 1800 60  0001 C CNN
 F 3 "" H 5700 1800 60  0000 C CNN
 	1    5700 1800
